Commit message: feat(sitl): configure 130g 15x15cm quadcopter physics with 1.5kg payload and full sensor suite (laser + 8x8 ToF + flow)

File: assets/chong_micro_quad.urdf (robot description, URDF)
Before this commit: robot chong_micro_quad, 6 links, 5 joints
Links:
- removed link arm_cross
- added link arm_cross_1, mass 0.005; visual box size=0.150 0.010 0.004
- added link arm_cross_2, mass 0.005; visual box size=0.150 0.010 0.004
- added link sensor_laser_down; visual cylinder length=0.008 radius=0.006
- added link sensor_optical_flow; visual box size=0.014 0.014 0.005
- added link sensor_tof_matrix; visual box size=0.008 0.020 0.012; visual cylinder length=0.002 radius=0.004
- link base_link: mass 0.033 -> 0.130; geometry collision box size=0.085 0.085 0.032; visual box size=0.050 0.050 0.006
- link rotor_1: mass 0.001 -> 0.003; geometry visual cylinder length=0.003 radius=0.040
- link rotor_2: mass 0.001 -> 0.003; geometry visual cylinder length=0.003 radius=0.040
- link rotor_3: mass 0.001 -> 0.003; geometry visual cylinder length=0.003 radius=0.040
- link rotor_4: mass 0.001 -> 0.003; geometry visual cylinder length=0.003 radius=0.040
Joints:
- removed joint base_to_arms
- added joint base_to_arm_1: type fixed, parent base_link, child arm_cross_1, origin xyz=0 0 0 rpy=0 0 0
- added joint base_to_arm_2: type fixed, parent base_link, child arm_cross_2, origin xyz=0 0 0 rpy=0 0 0
- added joint base_to_flow: type fixed, parent base_link, child sensor_optical_flow, origin xyz=-0.020 0.0 -0.017 rpy=0 0 0
- added joint base_to_laser: type fixed, parent base_link, child sensor_laser_down, origin xyz=0.0 0.0 -0.018 rpy=0 0 0
- added joint base_to_tof: type fixed, parent base_link, child sensor_tof_matrix, origin xyz=0.042 0.0 0.005 rpy=0 0 0
- joint joint_rotor_1: origin xyz=-0.0325 0.0325 0.006 rpy=0 0 0 -> xyz=-0.053 0.053 0.008 rpy=0 0 0
- joint joint_rotor_2: origin xyz=0.0325 0.0325 0.006 rpy=0 0 0 -> xyz=0.053 0.053 0.008 rpy=0 0 0
- joint joint_rotor_3: origin xyz=-0.0325 -0.0325 0.006 rpy=0 0 0 -> xyz=-0.053 -0.053 0.008 rpy=0 0 0
- joint joint_rotor_4: origin xyz=0.0325 -0.0325 0.006 rpy=0 0 0 -> xyz=0.053 -0.053 0.008 rpy=0 0 0
